File: hardware/4hp-diy-uncertainty/DIY Uncertainty.kicad_pcb (KiCad board)
At the start: 2 copper layers, 52.1 x 116.8 mm, 67 parts, among them J1 AudioJack2, J11 AudioJack2, J2 AudioJack2, J3 AudioJack2, J4 AudioJack2, J5 Conn_01x03_Pin, J6 AudioJack2, J7 AudioJack2, J8 AudioJack2, J9 AudioJack2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

Commit message: misc updates from kate
Connections:
- U2 pad 10: Net-(U1-2A) -> Net-(U1-3A)
- U2 pad 11: Net-(U1-1A) -> Net-(U1-4A)
- U2 pad 8: Net-(U1-4A) -> Net-(U1-1A)
- U2 pad 9: Net-(U1-3A) -> Net-(U1-2A)
- U4 pad 1: GND -> +3.3V
- U4 pad 2: +3.3V -> GND
- XJ8 pad 1: Net-(J9-Pad3) -> GND
- XJ8 pad 2: GND -> Net-(J9-Pad3)
Routing:
- net Net-(U1-4A): track 39.8 -> 47.4 mm
- net Net-(U1-1A): track 38.0 -> 30.7 mm
- net Net-(J9-Pad3): track 30.2 -> 33.2 mm
- net Net-(U1-2A): track 46.3 -> 43.8 mm
- net Net-(U5-2Y): track 51.1 -> 53.4 mm
- net +3.3V: track 44.3 -> 46.1 mm
- net Net-(J2-Pad3): track 55.1 -> 56.6 mm
- net Net-(U1-3A): track 50.0 -> 51.5 mm
- net Net-(U2-PA11_A3_D3): track 60.5 -> 61.4 mm
- net Net-(U2-PA10_A2_D2): track 64.7 -> 65.4 mm
- net Net-(U5-1Y): track 71.7 -> 72.4 mm
- net Net-(J5-Pin_2): track 11.4 -> 11.6 mm, vias 0 -> 1
- net Net-(J5-Pin_1): track 15.0 -> 15.1 mm, vias 0 -> 1
