File: hardware/4hp-diy-uncertainty/DIY Uncertainty.kicad_sch (KiCad schematic)
At the start: 47 parts, among them J1 AudioJack2, J11 AudioJack2, J2 AudioJack2, J3 AudioJack2, J4 AudioJack2, J5 Conn_01x03_Pin, J6 AudioJack2, J7 AudioJack2, J8 AudioJack2, J9 AudioJack2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

Commit message: misc updates from kate
Connections:
- net +3.3V: now also U4.1 (VO); no longer U4.2 (VO)
- net GND: now also U4.2 (GND); no longer U4.1 (GND)
- net at U2.10 (PA5_A9_D9_MISO): now also U1.9 (3A); no longer U1.5 (2A)
- net at U2.11 (PA6_A10_D10_MOSI): now also U1.12 (4A); no longer U1.2 (1A)
- net at U2.8 (PB09_A7_D7_RX): now also U1.2 (1A); no longer U1.12 (4A)
- net at U2.9 (PA7_A8_D8_SCK): now also U1.5 (2A); no longer U1.9 (3A)
